Commit message: added rps-to-thrust function, added measurement smoothing, added collected rps-to-thrust and throttle-to-rps data

File: arcs/code/data_collection/calibration/scenario/floor.urdf (robot description, URDF)
Before this commit: robot floor, 2 links, 1 joints
Links:
- link main: geometry collision box size=5.0 5.0 0.01; visual mesh filename=meshes/floor.stl scale=0.3 0.3 0.3

File: arcs/code/two-p600-experiments/floor.urdf (robot description, URDF)
Before this commit: robot floor, 2 links, 1 joints
Links:
- link main: geometry collision box size=5.0 5.0 0.01; visual mesh filename=meshes/floor.stl scale=0.5 0.5 0.5
